File: KiCad/KiCad.kicad_sch (KiCad schematic)
At the start: 51 parts, among them J1 DC-IN, J2 TYPE-C, J3 Conn_01x03_Pin, J4 Conn_01x03_Pin, J5 Conn_01x03_Pin, J6 Conn_01x03_Pin, Q1 IRF3708, SW1 reset, SW2 start, U1 ESP32-WROOM-32E, U2 MP1584EN, U3 CH340C, U4 RT9013-33GB, U5 DM-OLED096-636, U6 INA232AIDDFR, U7 MIC4420YM, U8 LM358

Commit message: 改以線圈溫升判斷安全電流，並讓上位機指定停測溫升。
分流改為 0.05 歐姆、測試負載 3 歐姆；電流碰到上限改走上一通過檔。同步整理機殼模型。

Co-authored-by: Cursor <cursoragent@cursor.com>
Parts:
- R8: value 0.1R -> 0.05R
Changed lines of the file:
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@@
 			)
 		)
-		(property "Value" "0.1R"
+		(property "Value" "0.05R"
 			(at 109.22 106.6799 0)
 			(effects
